File: double_comparator.kicad_pcb (KiCad board)
At the start: 4 copper layers, 36 parts, among them CON1 BNC_361V504EFT, CON2 BNC_361V504EFT, CON3 BNC_361V504EFT, CON4 BNC_361V504EFT, U4 ADCMP552

Commit message: updated design
Parts:
- removed C18, C21, C28, C29, C30, C34, C35: 100nF, carrier:C_MLCC_0603
- removed C19: 100n, carrier:C_MLCC_0603
- removed CON1, CON2, CON3, CON4: BNC_361V504EFT, carrier:BNC_V-BITE_PCB_EDGE
- removed R22, R23: DNP, carrier:R_0603
- removed R27, R28, R29, R30, R31, R32: 49.9, carrier:R_0603
- removed U4: ADCMP552, carrier:QSOP20
- added C10: 100nF, Capacitor_SMD:C_0603_1608Metric, F.Cu at (144.3, 65.8)
- added C12: 100nF, Capacitor_SMD:C_0603_1608Metric, F.Cu at (165.3, 61.7)
- added C13: 100nF, Capacitor_SMD:C_0603_1608Metric, F.Cu at (139.6, 61.5)
- added C3: 0.1uF, Capacitor_SMD:C_0603_1608Metric, F.Cu at (145.3, 76.2)
- added C4: 100nF, Capacitor_SMD:C_0603_1608Metric, F.Cu at (162.1, 73.4)
- added C5: 100nF, Capacitor_SMD:C_0603_1608Metric, F.Cu at (158.2, 72.9)
- added C6: 100nF, Capacitor_SMD:C_0603_1608Metric, F.Cu at (166.0, 82.1)
- added C7: 100nF, Capacitor_SMD:C_0603_1608Metric, F.Cu at (140.8, 82.0)
- added C8: 100nF, Capacitor_SMD:C_0603_1608Metric, F.Cu at (144.3, 64.0)
- added C9: 100nF, Capacitor_SMD:C_0603_1608Metric, F.Cu at (162.0, 64.3)
- added J1: Conn_01x02_Pin, Connector_Molex:Molex_KK-254_AE-6410-02A_1x02_P2.54mm_Vertical, F.Cu at (152.7, 61.5)
- added J2: Conn_Coaxial, local_footprints:BNC_V-BITE_PCB_EDGE, F.Cu at (137.2, 92.7)
- added J3: Conn_Coaxial, local_footprints:BNC_V-BITE_PCB_EDGE, F.Cu at (170.2, 92.7)
- added J4: Conn_Coaxial, local_footprints:BNC_V-BITE_PCB_EDGE, F.Cu at (170.2, 57.1)
- added J5: Conn_Coaxial, local_footprints:BNC_V-BITE_PCB_EDGE, F.Cu at (137.2, 57.1)
- added R10: DNP, Resistor_SMD:R_0603_1608Metric, F.Cu at (153.9, 79.3)
- added R14: 49.9, Resistor_SMD:R_0603_1608Metric, F.Cu at (147.1, 65.1)
- added R15: 49.9, Resistor_SMD:R_0603_1608Metric, F.Cu at (161.9, 62.7)
- added R16: 49.9, Resistor_SMD:R_0603_1608Metric, F.Cu at (159.7, 65.0)
- added R17: 1k, Resistor_SMD:R_0603_1608Metric, F.Cu at (141.5, 67.6)
- added R18: 1k, Resistor_SMD:R_0603_1608Metric, F.Cu at (141.5, 64.1)
- added R19: 1k, Resistor_SMD:R_0603_1608Metric, F.Cu at (164.3, 67.4)
- added R20: 1k, Resistor_SMD:R_0603_1608Metric, F.Cu at (164.3, 64.2)
- added U1: ADCMP552, Package_SO:QSOP-20_3.9x8.7mm_P0.635mm, F.Cu at (153.3, 73.1)
- C1: value 100nF -> 0.1uF; footprint carrier:C_MLCC_0603 -> Capacitor_SMD:C_0603_1608Metric
- C11: value 0.1u -> 100nF; footprint carrier:C_MLCC_0603 -> Capacitor_SMD:C_0603_1608Metric
- C2: footprint carrier:C_MLCC_0603 -> Capacitor_SMD:C_0603_1608Metric
- R1: value 1k -> 100; footprint carrier:R_0603 -> Resistor_SMD:R_0603_1608Metric
- R11, R12, R13: value 1k -> 49.9; footprint carrier:R_0603 -> Resistor_SMD:R_0603_1608Metric
- R2, R3, R6: footprint carrier:R_0603 -> Resistor_SMD:R_0603_1608Metric
- R4: value 1.1k -> 100; footprint carrier:R_0603 -> Resistor_SMD:R_0603_1608Metric
- R5: value 1k -> 1.1k; footprint carrier:R_0603 -> Resistor_SMD:R_0603_1608Metric
- R7: value 100 -> 1.1k; footprint carrier:R_0603 -> Resistor_SMD:R_0603_1608Metric
- R8: value 100 -> 1k; footprint carrier:R_0603 -> Resistor_SMD:R_0603_1608Metric
- R9: value 1.1k -> DNP; footprint carrier:R_0603 -> Resistor_SMD:R_0603_1608Metric
- moved C11 137.0 mm to (162.0, 65.8), turned to 0 degrees
- moved R3 119.7 mm to (159.6, 81.3), turned to 0 degrees
- moved R7 119.3 mm to (165.4, 73.1)
- moved R8 119.0 mm to (163.6, 73.5)
- moved R4 116.5 mm to (162.9, 81.3), turned to 0 degrees
- moved R13 115.5 mm to (158.2, 65.0)
- moved R1 110.6 mm to (146.6, 81.3), turned to 180 degrees
- moved C2 110.4 mm to (161.3, 83.6)
- moved R11 109.1 mm to (149.1, 65.1), turned to 90 degrees
- moved C1 106.0 mm to (145.0, 83.6)
- moved R2 105.9 mm to (143.6, 81.3), turned to 180 degrees
- moved R12 104.5 mm to (144.3, 62.2), turned to 180 degrees
- moved R9 104.2 mm to (152.4, 79.3)
- moved R5 103.8 mm to (142.2, 73.1), turned to -90 degrees
- moved R6 100.9 mm to (142.2, 76.1)
Routing:
- net -3V3: track 0.00 -> 119.7 mm, vias 0 -> 8
- net Net-(J5-In): track 0.00 -> 18.1 mm
- net Net-(J4-In): track 0.00 -> 17.7 mm
- net Net-(J2-In): track 0.00 -> 17.1 mm
- net Net-(J3-In): track 0.00 -> 16.7 mm
- net DGND: track 3.80 -> 19.7 mm, vias 0 -> 11
- net VCCIO_34: track 14.8 -> 0.00 mm
- net /Comparators/TH1: track 13.6 -> 0.00 mm
- net /Comparators/TH2: track 12.0 -> 0.00 mm
- net /INPUT1: track 0.00 -> 11.8 mm
- net /TH1: track 0.00 -> 10.5 mm
- net /TH2: track 0.00 -> 10.2 mm
- net OUT1_N: track 0.00 -> 9.82 mm
- net OUT2_N: track 0.00 -> 9.42 mm
- net Net-(C8-Pad1): track 0.00 -> 7.49 mm
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- added copper zone on B.Cu, net DGND
- added copper zone on F.Cu, net DGND
Other:
- copper layers 4 -> 2

Commit message: version ready to be printed
Parts:
- added H1: MountingHole, MountingHole:MountingHole_3mm, F.Cu at (181.6, 55.9)
- added H2: MountingHole, MountingHole:MountingHole_3mm, F.Cu at (125.7, 94.0)
- added H3: MountingHole, MountingHole:MountingHole_3mm, F.Cu at (125.7, 55.9)
- added H4: MountingHole, MountingHole:MountingHole_3mm, F.Cu at (181.6, 94.0)
- moved C7 7.19 mm to (145.0, 76.2), turned to 90 degrees
- moved C6 7.12 mm to (161.3, 76.7), turned to 90 degrees
- moved R1 5.87 mm to (147.4, 75.4), turned to 0 degrees
- moved R2 5.69 mm to (147.4, 77.0)
- moved R4 5.52 mm to (158.9, 77.5)
- moved R6 5.49 mm to (146.8, 73.1), turned to 90 degrees
- moved R3 5.47 mm to (158.9, 75.9), turned to 180 degrees
- moved C1 5.25 mm to (148.3, 79.4)
- moved C2 4.86 mm to (158.1, 79.9)
- moved C3 4.49 mm to (148.6, 73.1), turned to -90 degrees
- moved R5 2.79 mm to (145.0, 73.1)
- moved C12 2.52 mm to (163.3, 60.2), turned to 90 degrees
- moved C13 1.97 mm to (141.5, 60.9)
- moved R9 0.98 mm to (151.6, 78.7), turned to 180 degrees
- moved R10 0.98 mm to (154.7, 78.7), turned to 180 degrees
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Routing:
- net /INPUT1: track 11.8 -> 5.70 mm
- net -3V3: track 119.7 -> 114.1 mm, vias 8 -> 4
- net /TH1: track 10.5 -> 5.93 mm
- net DGND: track 19.7 -> 24.0 mm, vias 11 -> 8
- net Net-(J3-In): track 16.7 -> 20.3 mm
- net /INPUT2: track 2.92 -> 5.68 mm
- net Net-(J5-In): track 18.1 -> 16.3 mm
- net Net-(J2-In): track 17.1 -> 18.9 mm
- net /TH2: track 10.2 -> 9.64 mm
- added copper zone on F.Cu, net -3V3
Other:
- board outline added: 66 x 48.3 mm
