File: double_comparator.kicad_sch (KiCad schematic)
At the start: 37 parts, among them CON1 BNC_361V504EFT, CON2 BNC_361V504EFT, CON3 BNC_361V504EFT, CON4 BNC_361V504EFT, J1 Conn_01x02_Pin, U1 ADCMP552

Commit message: updated design
Parts:
- removed C1: 0.1u, carrier:C_MLCC_0603, symbol carrier-eagle-import:C_MLCC_SMDCMLCC_0603
- removed C10, C11, C3, C4, C5, C6, C7, C8, C9: 100nF, carrier:C_MLCC_0603, symbol carrier-eagle-import:C_MLCC_SMDCMLCC_0603
- removed C2: 100n, carrier:C_MLCC_0603, symbol carrier-eagle-import:C_MLCC_SMDCMLCC_0603
- removed CON1, CON2, CON3, CON4: BNC_361V504EFT, carrier:BNC_V-BITE_PCB_EDGE, symbol carrier-eagle-import:BNC_361V504EFT
- removed R1, R2, R3, R4: 100, carrier:R_0603, symbol carrier-eagle-import:R_SMDR0603
- removed R10, R9: DNP, carrier:R_0603, symbol carrier-eagle-import:R_SMDR0603
- removed R11, R12, R13, R14, R15, R16: 49.9, carrier:R_0603, symbol carrier-eagle-import:R_SMDR0603
- removed R17, R18, R19, R20, R8: 1k, carrier:R_0603, symbol carrier-eagle-import:R_SMDR0603
- removed R5, R6, R7: 1.1k, carrier:R_0603, symbol carrier-eagle-import:R_SMDR0603
- added C1, C3: 0.1uF, Capacitor_SMD:C_0603_1608Metric, symbol Device:C
- added C10, C11, C12, C13, C2, C4, C5, C6, C7, C8, C9: 100nF, Capacitor_SMD:C_0603_1608Metric, symbol Device:C
- added J2, J3, J4, J5: Conn_Coaxial, local_footprints:BNC_V-BITE_PCB_EDGE, symbol Connector:Conn_Coaxial
- added R1, R2, R3, R4: 100, Resistor_SMD:R_0603_1608Metric, symbol Device:R_US
- added R10, R9: DNP, Resistor_SMD:R_0603_1608Metric, symbol Device:R_US
- added R11, R12, R13, R14, R15, R16: 49.9, Resistor_SMD:R_0603_1608Metric, symbol Device:R_US
- added R17, R18, R19, R20, R8: 1k, Resistor_SMD:R_0603_1608Metric, symbol Device:R_US
- added R5, R6, R7: 1.1k, Resistor_SMD:R_0603_1608Metric, symbol Device:R_US
- U1: footprint carrier:QSOP20 -> Package_SO:QSOP-20_3.9x8.7mm_P0.635mm
Connections:
- net -3V3: now also C12.1, C13.1, C3.1, C4.2, C5.1, C6.1, C7.1, C8.2, C9.2, R10.2, R12.2, R15.2, R18.2, R2.2, R20.2, R4.2, R6.2, R8.2, R9.1; no longer J1.1 (Pin_1), U1.1 (VCCO1), U1.17 (VCCO17), U1.20 (VCCO20), U1.4 (VCCO4), U1.7 (VCCI7)
- net INPUT1: now also C1.2, R1.2, R2.1
- net INPUT2: now also C2.2, R3.2, R4.1
- net OUT1_N: now also C10.1, R14.1
- net OUT1_P: now also R11.1
- net OUT2_N: now also C11.1, R16.1
- net OUT2_P: now also R13.1
- net TH1: now also C3.2, R5.2, R6.1
- net TH2: now also C4.1, R7.2, R8.1
- net at U1.11 (HYSB): now also R10.1
- net at U1.10 (HYSA): now also R9.2
- new net: C2.1, J3.1 (In)
- new net: C8.1, R11.2, R12.1, R14.2
- new net: C11.2, J4.1 (In), R19.2, R20.1
- new net: C10.2, J5.1 (In), R17.2, R18.1
- new net: C9.1, R13.2, R15.1, R16.2
- new net: C1.1, J2.1 (In)
- new net DGND: C12.2, C13.2, C5.2, C6.2, C7.2, J1.1 (Pin_1), J2.2 (Ext), J3.2 (Ext), J4.2 (Ext), J5.2 (Ext), R1.1, R17.1, R19.1, R3.1, R5.1, R7.1, U1.1 (VCCO1), U1.17 (VCCO17), U1.20 (VCCO20), U1.4 (VCCO4), U1.7 (VCCI7)

Commit message: version ready to be printed
Parts:
- added H1, H2, H3, H4: MountingHole, MountingHole:MountingHole_3mm, symbol Mechanical:MountingHole
Changed lines of the file:
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@@
+    )
+  )
+  (symbol (lib_id "Mechanical:MountingHole") (at 133.35 161.29 0) (unit 1)
+    (in_bom yes) (on_board yes) (dnp no) (fields_autoplaced)
+    (property "Reference" "H3" (at 135.89 160.02 0)
+      (effects (font (size 1.27 1.27)) (justify left))
+    )
+    (property "Value" "MountingHole" (at 135.89 162.56 0)
+      (effects (font (size 1.27 1.27)) (justify left))
+    )
+    (property "Footprint" "MountingHole:MountingHole_3mm" (at 133.35 161.29 0)
+      (effects (font (size 1.27 1.27)) hide)
+    )
+    (property "Datasheet" "~" (at 133.35 161.29 0)
+      (effects (font (size 1.27 1.27)) hide)
+    )
+    (instances
+      (project "double_comparator"
+        (path "/ffd175d1-912a-4224-be1e-a8198680f46b"
+          (reference "H3") (unit 1)
+        )
+      )
     )
   )
@@
     )
   )
+  (symbol (lib_id "Mechanical:MountingHole") (at 154.94 152.4 0) (unit 1)
+    (in_bom yes) (on_board yes) (dnp no) (fields_autoplaced)
+    (property "Reference" "H2" (at 157.48 151.13 0)
+      (effects (font (size 1.27 1.27)) (justify left))
+    )
+    (property "Value" "MountingHole" (at 157.48 153.67 0)
+      (effects (font (size 1.27 1.27)) (justify left))
+    )
+    (property "Footprint" "MountingHole:MountingHole_3mm" (at 154.94 152.4 0)
+      (effects (font (size 1.27 1.27)) hide)
+    )
+    (property "Datasheet" "~" (at 154.94 152.4 0)
+      (effects (font (size 1.27 1.27)) hide)
+    )
+    (instances
+      (project "double_comparator"
+        (path "/ffd175d1-912a-4224-be1e-a8198680f46b"
+          (reference "H2") (unit 1)
+        )
+      )
+    )
+  )
   (symbol (lib_id "Connector:Conn_Coaxial") (at 280.67 129.54 0) (unit 1)
     (in_bom yes) (on_board yes) (dnp no)
@@
     )
   )
+  (symbol (lib_id "Mechanical:MountingHole") (at 154.94 161.29 0) (unit 1)
+    (in_bom yes) (on_board yes) (dnp no) (fields_autoplaced)
+    (property "Reference" "H4" (at 157.48 160.02 0)
+      (effects (font (size 1.27 1.27)) (justify left))
+    )
+    (property "Value" "MountingHole" (at 157.48 162.56 0)
+      (effects (font (size 1.27 1.27)) (justify left))
+    )
+    (property "Footprint" "MountingHole:MountingHole_3mm" (at 154.94 161.29 0)
+      (effects (font (size 1.27 1.27)) hide)
+    )
+    (property "Datasheet" "~" (at 154.94 161.29 0)
+      (effects (font (size 1.27 1.27)) hide)
+    )
+    (instances
+      (project "double_comparator"
+        (path "/ffd175d1-912a-4224-be1e-a8198680f46b"
+          (reference "H4") (unit 1)
+        )
+      )
+    )
+  )
   (symbol (lib_id "Connector:Conn_Coaxial") (at 15.24 127 0) (mirror y) (unit 1)
     (in_bom yes) (on_board yes) (dnp no)
@@
         )
       )
+    )
+  )
+  (symbol (lib_id "Mechanical:MountingHole") (at 133.35 152.4 0) (unit 1)
+    (in_bom yes) (on_board yes) (dnp no) (fields_autoplaced)
+    (property "Reference" "H1" (at 135.89 151.13 0)
+      (effects (font (size 1.27 1.27)) (justify left))
+    )
+    (property "Value" "MountingHole" (at 135.89 153.67 0)
+      (effects (font (size 1.27 1.27)) (justify left))
+    )
+    (property "Footprint" "MountingHole:MountingHole_3mm" (at 133.35 152.4 0)
+      (effects (font (size 1.27 1.27)) hide)
+    )
+    (property "Datasheet" "~" (at 133.35 152.4 0)
+      (effects (font (size 1.27 1.27)) hide)
+    )
+    (instances
+      (project "double_comparator"
+        (path "/ffd175d1-912a-4224-be1e-a8198680f46b"
+          (reference "H1") (unit 1)
+        )
+      )
